File: KiCad/L86/L86.kicad_pcb (KiCad board)
At the start: 2 copper layers, 38.5 x 30 mm, 4 parts, among them J1 Conn_01x06, U1 L86-M33, U2 QR

Commit message: SIlkscreen
Parts:
- moved Logo1 0.28 mm to (99.4, 95.4)
Other:
- board text added: "BAT"
- board text added: "GND"
- board text added: "PPS"
- board text added: "VCC"
- board text added: "←TX"
- board text added: "→RX"
Changed lines of the file:
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@@
   )
   (footprint "RevK:AJK" (layer "B.Cu")
-    (at 99.4 95.1 180)
+    (at 99.4 95.375 180)
     (property "Note" "Non part, PCB printed")
     (property "Sheetfile" "L86.kicad_sch")
@@
   (gr_line (start 85 113) (end 85 87) (layer "Edge.Cuts") (width 0.1))
   (gr_line (start 123.5 91) (end 123.5 109) (layer "Edge.Cuts") (width 0.1))
+  (gr_text "→RX" (at 120.5 106.25) (layer "B.SilkS")
+    (effects (font (size 1 1) (thickness 0.15)) (justify mirror))
+  )
+  (gr_text "BAT" (at 120.5 96.25) (layer "B.SilkS")
+    (effects (font (size 1 1) (thickness 0.15)) (justify mirror))
+  )
+  (gr_text "←TX" (at 120.5 103.75) (layer "B.SilkS")
+    (effects (font (size 1 1) (thickness 0.15)) (justify mirror))
+  )
+  (gr_text "GND" (at 120.5 101.25) (layer "B.SilkS")
+    (effects (font (size 1 1) (thickness 0.15)) (justify mirror))
+  )
+  (gr_text "VCC" (at 120.5 98.75) (layer "B.SilkS")
+    (effects (font (size 1 1) (thickness 0.15)) (justify mirror))
+  )
+  (gr_text "PPS" (at 120.5 93.75) (layer "B.SilkS")
+    (effects (font (size 1 1) (thickness 0.15)) (justify mirror))
+  )
   (segment (start 106 106.25) (end 107.65 106.25) (width 0.25) (layer "F.Cu") (net 8))
   (segment (start 107.65 106.25) (end 107.75 106.35) (width 0.25) (layer "F.Cu") (net 8))
