File: KiCad/L86.kicad_sch (KiCad schematic)
At the start: 4 parts, among them J1 Conn_01x06, U1 L86-M33, U2 QR

Commit message: Clean up
Connections:
- no-connect marks 0 -> 5
Other:
- moved on the sheet: U1
Changed lines of the file:
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@@
   (junction (at 149.86 73.66) (diameter 0) (color 0 0 0 0)
   )
+  (no_connect (at 116.84 68.58))
+  (no_connect (at 116.84 66.04))
+  (no_connect (at 116.84 73.66))
+  (no_connect (at 116.84 76.2))
+  (no_connect (at 116.84 78.74))
   (wire (pts (xy 147.32 73.66) (xy 149.86 73.66))
     (stroke (width 0) (type default) (color 0 0 0 0))
@@
     )
   )
-  (symbol (lib_id "RevK:L86-M33") (at 133.35 72.39 0) (unit 1)
+  (symbol (lib_id "RevK:L86-M33") (at 132.08 72.39 0) (unit 1)
     (in_bom yes) (on_board yes) (fields_autoplaced)
-    (property "Reference" "U1" (id 0) (at 132.715 58.581 0))
-    (property "Value" "L86-M33" (id 1) (at 132.715 61.1179 0))
-    (property "Footprint" "RevK:L86-M33" (id 2) (at 138.43 71.12 0)
+    (property "Reference" "U1" (id 0) (at 131.445 58.581 0))
+    (property "Value" "L86-M33" (id 1) (at 131.445 61.1179 0))
+    (property "Footprint" "RevK:L86-M33" (id 2) (at 137.16 71.12 0)
       (effects (font (size 1.27 1.27)) hide)
     )
-    (property "Datasheet" "" (id 3) (at 138.43 71.12 0)
+    (property "Datasheet" "" (id 3) (at 137.16 71.12 0)
       (effects (font (size 1.27 1.27)) hide)
     )
