File: KiCad/Display.kicad_pcb (KiCad board)
At the start: 2 copper layers, 44.5 x 67 mm, 30 parts, among them J1 DC, J2 USB-C, M1 OLED1.5-RGB, U1 L86-M33, U2 ESP32-PICO-MINI-02, U3 FT231XQ, U4 LMR16006+FB, U5 QR

Commit message: Library update
Routing:
- net TICK: track 35.2 -> 49.2 mm
- net +3V3: track 119.7 -> 127.9 mm
- net GND: track 25.5 -> 26.5 mm
Other:
- board text added: "13"
- board text added: "14"
- board text added: "26"
- board text added: "27"
- board text added: "3.3"
- board text added: "8"
- board text added: "DC 4V-60V"
- board text added: "GPS Display"
- board text added: "LED: 21/22/19 GPSTICK: 33 GPSRX: 32 GPSTX: 25"
- board text added: "⏚"

Commit message: DRC tweaks
Parts:
- D1: footprint Diode_SMD:D_1206_3216Metric -> RevK:D_1206
Other:
- outline, holes or cut-outs redrawn
- rule pad_to_mask_clearance: 0 -> 0.01

Commit message: Resistors
Parts:
- R12: value 3M 1% or NF -> 30k 1% or NF
- R8: value 10M 1% or 0R -> 100k 1% or 0R
