File: KiCad/Display.kicad_sch (KiCad schematic)
At the start: 36 parts, among them J1 DC, J2 I/O, J3 USB-C, U1 ESP32-PICO-MINI-02, U2 L96-M33, U3 FT231XQ, U4 LMR16006+FB, U5 QR

Commit message: Started on Display board.
Parts:
- removed J2: I/O, RevK:Molex_MiniSPOX_H6RA, symbol Connector_Generic:Conn_01x06
- removed JP1: IO6, RevK:Pad_1206_0805_Open, symbol Jumper:Jumper_2_Open
- removed JP2: IO4, RevK:Pad_1206_0805_Open, symbol Jumper:Jumper_2_Open
- removed JP3: IO3, RevK:Pad_1206_0805_Open, symbol Jumper:Jumper_2_Open
- removed JP4: IO1, RevK:Pad_1206_0805_Open, symbol Jumper:Jumper_2_Open
- removed JP5: IO6, RevK:Pad_1206_0805_Bridged, symbol Jumper:Jumper_2_Bridged
- removed JP6: IO3, RevK:Pad_1206_0805_Bridged, symbol Jumper:Jumper_2_Bridged
- removed R6: 470K, RevK:R_0603, symbol Device:R
- removed R7: 100K, RevK:R_0603, symbol Device:R
- removed U2: L96-M33, RevK:L96-M33, symbol RevK:L96-M33
- added BT1: Battery_Cell, Battery:BatteryHolder_Keystone_3002_1x2032, symbol Device:Battery_Cell
- added M1: OLED1.5-RGB, RevK:OLED1.5-RGB, symbol RevK:OLED1.5-RGB
- added R4, R5: 27R, RevK:R_0603, symbol Device:R
- added U1: L86-M33, RevK:L86-M33, symbol RevK:L86-M33
- renumbered J3 to J2, R4 to R6, R5 to R7, U1 to U2
Connections:
- net GPSRST is gone; now on net TICK: U2.13 (IO33)
- net +3V3: now also M1.1 (Vcc), U1.4 (VCC)
- net B: now also U2.35 (IO21); no longer U2.33 (IO19)
- net D+: now also R5.2; no longer J2.A6 (D+), J2.B6 (D+)
- net D-: now also R4.2; no longer J2.A7 (D-), J2.B7 (D-)
- net G: now also U2.33 (IO19); no longer U2.34 (IO22)
- net GND: now also BT1.2 (-), M1.2 (GND), M1.S (SCREWS), U1.12 (GND), U1.3 (GND)
- net GPSRX: now also U2.12 (IO32), U1.1 (RXD1); no longer U2.16 (IO26)
- net GPSTX: now also U1.2 (TXD1)
- net R: now also U2.34 (IO22); no longer U2.35 (IO21)
- net TICK: now also U1.6 (1PPS); no longer U2.18 (IO14)
- net BAT: no longer names the net of U2.9 (I34)
- net GPSON: no longer names the net of U2.17 (IO27)
- net IO1 renamed OLED-RST
- net OLED-RST: now also M1.7 (RST)
- net IO2: no longer names the net of U2.26 (IO20)
- net IO3: no longer names the net of U2.24 (IO4)
- net IO4: no longer names the net of U2.27 (IO7)
- net IO5 renamed OLED-MOSI
- net OLED-MOSI: now also M1.3 (DIN)
- net IO6 renamed OLED-CS0
- net OLED-CS0: now also M1.5 (CS)
- new net: J2.A6 (D+), J2.B6 (D+), R5.1
- new net: J2.A7 (D-), J2.B7 (D-), R4.1
- new net: BT1.1 (+), U1.5 (V_BKCP)
- new net OLED-DC: M1.6 (DC), U2.18 (IO14)
- new net OLED-SCLK: M1.4 (CLK), U2.16 (IO26)
- no-connect marks 20 -> 18
Other:
- note removed: "Ext passive is 100pF series"
- note removed: "Open"
- note removed: "Open or VCC"
- title: GPS / Glider control board -> GPS reference
- moved on the sheet: D1, J2, R2, R3

Commit message: Tracked, needs tidying
Connections:
- no-connect marks 18 -> 20
Changed lines of the file:
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@@
   (no_connect (at 81.28 71.12))
   (no_connect (at 50.8 50.8))
+  (no_connect (at 50.8 78.74))
+  (no_connect (at 50.8 83.82))
   (no_connect (at 185.42 116.84))
   (no_connect (at 185.42 119.38))

Commit message: tracked
Connections:
- net B: now also U2.33 (IO19); no longer U2.35 (IO21)
- net G: now also U2.34 (IO22); no longer U2.33 (IO19)
- net OLED-CS0: now also U2.17 (IO27); no longer U2.20 (IO13)
- net OLED-RST: now also U2.20 (IO13); no longer U2.21 (IO15)
- net R: now also U2.35 (IO21); no longer U2.34 (IO22)
- no-connect marks 20 -> 19
Changed lines of the file:
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@@
   (no_connect (at 185.42 114.3))
   (no_connect (at 50.8 73.66))
-  (no_connect (at 81.28 83.82))
   (no_connect (at 48.26 139.7))
   (no_connect (at 48.26 142.24))
@@
     )
   )
-  (global_label "OLED-RST" (shape output) (at 50.8 91.44 180) (fields_autoplaced)
-    (effects (font (size 1.27 1.27)) (justify right))
-    (property "Intersheet References" "${INTERSHEET_REFS}" (id 0) (at 38.6787 91.3606 0)
+  (global_label "OLED-RST" (shape output) (at 50.8 86.36 180) (fields_autoplaced)
+    (effects (font (size 1.27 1.27)) (justify right))
+    (property "Intersheet References" "${INTERSHEET_REFS}" (id 0) (at 38.6787 86.2806 0)
       (effects (font (size 1.27 1.27)) (justify right) hide)
     )
@@
     )
   )
-  (global_label "R" (shape input) (at 81.28 76.2 0) (fields_autoplaced)
-    (effects (font (size 1.27 1.27)) (justify left))
-    (property "Intersheet References" "${INTERSHEET_REFS}" (id 0) (at -3.175 -16.51 0)
-      (effects (font (size 1.27 1.27)) hide)
+  (global_label "R" (shape output) (at 81.28 73.66 0) (fields_autoplaced)
+    (effects (font (size 1.27 1.27)) (justify left))
+    (property "Intersheet References" "${INTERSHEET_REFS}" (id 0) (at 84.8742 73.5806 0)
+      (effects (font (size 1.27 1.27)) (justify left) hide)
     )
   )
@@
     )
   )
-  (global_label "OLED-CS0" (shape output) (at 50.8 86.36 180) (fields_autoplaced)
-    (effects (font (size 1.27 1.27)) (justify right))
-    (property "Intersheet References" "${INTERSHEET_REFS}" (id 0) (at 38.4368 86.2806 0)
-      (effects (font (size 1.27 1.27)) (justify right) hide)
+  (global_label "OLED-CS0" (shape output) (at 81.28 83.82 0) (fields_autoplaced)
+    (effects (font (size 1.27 1.27)) (justify left))
+    (property "Intersheet References" "${INTERSHEET_REFS}" (id 0) (at 93.6432 83.8994 0)
+      (effects (font (size 1.27 1.27)) (justify left) hide)
     )
   )
@@
     )
   )
-  (global_label "G" (shape input) (at 81.28 68.58 0) (fields_autoplaced)
-    (effects (font (size 1.27 1.27)) (justify left))
-    (property "Intersheet References" "${INTERSHEET_REFS}" (id 0) (at -3.175 -19.05 0)
-      (effects (font (size 1.27 1.27)) hide)
+  (global_label "G" (shape output) (at 81.28 76.2 0) (fields_autoplaced)
+    (effects (font (size 1.27 1.27)) (justify left))
+    (property "Intersheet References" "${INTERSHEET_REFS}" (id 0) (at 84.8742 76.1206 0)
+      (effects (font (size 1.27 1.27)) (justify left) hide)
     )
   )
@@
     )
   )
-  (global_label "B" (shape input) (at 81.28 73.66 0) (fields_autoplaced)
-    (effects (font (size 1.27 1.27)) (justify left))
-    (property "Intersheet References" "${INTERSHEET_REFS}" (id 0) (at -3.175 -21.59 0)
-      (effects (font (size 1.27 1.27)) hide)
-    )
-  )
+  (global_label "B" (shape output) (at 81.28 68.58 0) (fields_autoplaced)
+    (effects (font (size 1.27 1.27)) (justify left))
+    (property "Intersheet References" "${INTERSHEET_REFS}" (id 0) (at 84.8742 68.5006 0)
+      (effects (font (size 1.27 1.27)) (justify left) hide)
+    )
+  )

Commit message: Clean up
Parts:
- removed Logo1: AA, RevK:AA, symbol RevK:AA
- J1: footprint RevK:Molex_MiniSPOX_H2RA -> RevK:DC
Connections:
- net GND: no longer M1.S (SCREWS)
Changed lines of the file:
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@@
     (pin "2")
-  )
-  (symbol (lib_id "RevK:AA") (at 266.7 172.72 0) (unit 1)
-    (in_bom no) (on_board yes)
-    (property "Reference" "Logo1" (id 0) (at 266.7 172.72 0)
-      (effects (font (size 1.27 1.27)) hide)
-    )
-    (property "Value" "AA" (id 1) (at 267.335 172.72 0)
-      (effects (font (size 1.27 1.27)) (justify left))
-    )
-    (property "Footprint" "RevK:AA" (id 2) (at 266.7 172.72 0)
-      (effects (font (size 1.27 1.27)) hide)
-    )
-    (property "Datasheet" "" (id 3) (at 266.7 172.72 0)
-      (effects (font (size 1.27 1.27)) hide)
-    )
-    (property "Note" "Non part, PCB printed" (id 4) (at 266.7 172.72 0)
-      (effects (font (size 1.27 1.27)) hide)
-    )
   )
   (symbol (lib_id "RevK:USB-C") (at 159.385 45.72 0) (unit 1)
@@
     (pin "2")
   )
-  (symbol (lib_id "RevK:OLED1.5-RGB") (at 231.14 109.22 0) (unit 1)
-    (in_bom yes) (on_board yes) (fields_autoplaced)
-    (property "Reference" "M1" (id 0) (at 263.525 118.5453 0)
-      (effects (font (size 1.27 1.27)) (justify left))
-    )
-    (property "Value" "OLED1.5-RGB" (id 1) (at 263.525 121.0822 0)
-      (effects (font (size 1.27 1.27)) (justify left))
-    )
-    (property "Footprint" "RevK:OLED1.5-RGB" (id 2) (at 250.19 132.08 0)
-      (effects (font (size 1.27 1.27)) hide)
-    )
-    (property "Datasheet" "" (id 3) (at 231.14 106.68 0)
+  (symbol (lib_id "RevK:OLED1.5-RGB") (at 231.14 106.68 0) (unit 1)
+    (in_bom yes) (on_board yes) (fields_autoplaced)
+    (property "Reference" "M1" (id 0) (at 263.525 116.0053 0)
+      (effects (font (size 1.27 1.27)) (justify left))
+    )
+    (property "Value" "OLED1.5-RGB" (id 1) (at 263.525 118.5422 0)
+      (effects (font (size 1.27 1.27)) (justify left))
+    )
+    (property "Footprint" "RevK:OLED1.5-RGB" (id 2) (at 250.19 129.54 0)
+      (effects (font (size 1.27 1.27)) hide)
+    )
+    (property "Datasheet" "" (id 3) (at 231.14 104.14 0)
       (effects (font (size 1.27 1.27)) hide)
     )
@@
     (pin "6")
     (pin "7")
-    (pin "S")
   )
   (symbol (lib_id "Device:R") (at 196.85 125.73 0) (unit 1)
@@
     (property "Reference" "J1" (id 0) (at 121.92 129.6502 0))
     (property "Value" "DC" (id 1) (at 121.92 132.1871 0))
-    (property "Footprint" "RevK:Molex_MiniSPOX_H2RA" (id 2) (at 121.92 132.08 0)
+    (property "Footprint" "RevK:DC" (id 2) (at 121.92 132.08 0)
       (effects (font (size 1.27 1.27)) hide)
     )
@@
     (pin "1")
     (pin "2")
-  )
-  (symbol (lib_id "power:GND") (at 231.14 129.54 270) (unit 1)
-    (in_bom yes) (on_board yes) (fields_autoplaced)
-    (property "Reference" "#PWR025" (id 0) (at 224.79 129.54 0)
-      (effects (font (size 1.27 1.27)) hide)
-    )
-    (property "Value" "GND" (id 1) (at 227.9651 129.9738 90)
-      (effects (font (size 1.27 1.27)) (justify right))
-    )
-    (property "Footprint" "" (id 2) (at 231.14 129.54 0)
-      (effects (font (size 1.27 1.27)) hide)
-    )
-    (property "Datasheet" "" (id 3) (at 231.14 129.54 0)
-      (effects (font (size 1.27 1.27)) hide)
-    )
-    (pin "1")
   )
   (symbol (lib_id "RevK:AJK") (at 274.32 173.355 0) (unit 1)
@@
       (reference "#PWR024") (unit 1) (value "GND") (footprint "")
     )
-    (path "/72c68ce1-de2f-4610-adad-51a6d09253a2"
-      (reference "#PWR025") (unit 1) (value "GND") (footprint "")
-    )
     (path "/392f7038-6e6c-4213-89de-22a308ba35ac"
       (reference "#PWR026") (unit 1) (value "GND") (footprint "")
@@
     )
     (path "/6632bf4c-766d-4d12-b7a8-80288e5f09e3"
-      (reference "J1") (unit 1) (value "DC") (footprint "RevK:Molex_MiniSPOX_H2RA")
+      (reference "J1") (unit 1) (value "DC") (footprint "RevK:DC")
     )
     (path "/00000000-0000-0000-0000-000060cc7ad1"
@@
       (reference "L1") (unit 1) (value "6.8uH") (footprint "RevK:Hidden")
     )
-    (path "/00000000-0000-0000-0000-000060b9351c"
-      (reference "Logo1") (unit 1) (value "AA") (footprint "RevK:AA")
-    )
     (path "/7fa098fb-b644-4e64-920e-8328b5d12f21"

Commit message: New battery holder
Parts:
- BT1: footprint Battery:BatteryHolder_Keystone_3002_1x2032 -> RevK:Battery-Holder-2032
- J1: footprint RevK:DC -> RevK:Molex_MiniSPOX_H2RA
Changed lines of the file:
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@@
     (property "Reference" "J1" (id 0) (at 121.92 129.6502 0))
     (property "Value" "DC" (id 1) (at 121.92 132.1871 0))
-    (property "Footprint" "RevK:DC" (id 2) (at 121.92 132.08 0)
+    (property "Footprint" "RevK:Molex_MiniSPOX_H2RA" (id 2) (at 121.92 132.08 0)
       (effects (font (size 1.27 1.27)) hide)
     )
@@
       (effects (font (size 1.27 1.27)) (justify left))
     )
-    (property "Footprint" "Battery:BatteryHolder_Keystone_3002_1x2032" (id 2) (at 99.06 145.796 90)
-      (effects (font (size 1.27 1.27)) hide)
-    )
-    (property "Datasheet" "~" (id 3) (at 99.06 145.796 90)
+    (property "Footprint" "RevK:Battery-Holder-2032" (id 2) (at 99.06 145.796 90)
+      (effects (font (size 1.27 1.27)) hide)
+    )
+    (property "Datasheet" "https://www.mouser.co.uk/datasheet/2/238/LNNC_S_A0002913840_1-2550745.pdf" (id 3) (at 99.06 145.796 90)
       (effects (font (size 1.27 1.27)) hide)
     )
@@
     )
     (path "/d2acb68c-44d4-4480-8eda-51e505a3f6f6"
-      (reference "BT1") (unit 1) (value "Battery_Cell") (footprint "Battery:BatteryHolder_Keystone_3002_1x2032")
+      (reference "BT1") (unit 1) (value "Battery_Cell") (footprint "RevK:Battery-Holder-2032")
     )
     (path "/00000000-0000-0000-0000-000060910a6c"
@@
     )
     (path "/6632bf4c-766d-4d12-b7a8-80288e5f09e3"
-      (reference "J1") (unit 1) (value "DC") (footprint "RevK:DC")
+      (reference "J1") (unit 1) (value "DC") (footprint "RevK:Molex_MiniSPOX_H2RA")
     )
     (path "/00000000-0000-0000-0000-000060cc7ad1"
