File: KiCad/Display.kicad_sch (KiCad schematic)
At the start: 30 parts, among them J1 DC, J2 USB-C, M1 OLED1.5-RGB, U1 L86-M33, U2 ESP32-PICO-MINI-02, U3 FT231XQ, U4 LMR16006+FB, U5 QR

Commit message: DRC tweaks
Parts:
- D1: footprint Diode_SMD:D_1206_3216Metric -> RevK:D_1206
Changed lines of the file:
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@@
     (property "Reference" "D1" (id 0) (at 193.675 24.9682 0))
     (property "Value" "D" (id 1) (at 193.675 27.2796 0))
-    (property "Footprint" "Diode_SMD:D_1206_3216Metric" (id 2) (at 193.675 30.48 0)
+    (property "Footprint" "RevK:D_1206" (id 2) (at 193.675 30.48 0)
       (effects (font (size 1.27 1.27)) hide)
     )
@@
     )
     (path "/00000000-0000-0000-0000-000060fbba89"
-      (reference "D1") (unit 1) (value "D") (footprint "Diode_SMD:D_1206_3216Metric")
+      (reference "D1") (unit 1) (value "D") (footprint "RevK:D_1206")
     )
     (path "/00000000-0000-0000-0000-000060ce13c1"

Commit message: Resistors
Parts:
- R12: value 3M 1% or NF -> 30k 1% or NF
- R8: value 10M 1% or 0R -> 100k 1% or 0R
Changed lines of the file:
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@@
       (effects (font (size 1.27 1.27)) (justify left))
     )
-    (property "Value" "10M 1% or 0R" (id 1) (at 236.855 46.355 90)
+    (property "Value" "100k 1% or 0R" (id 1) (at 236.855 46.355 90)
       (effects (font (size 1.27 1.27)) (justify left))
     )
@@
       (effects (font (size 1.27 1.27)) (justify right))
     )
-    (property "Value" "3M 1% or NF" (id 1) (at 241.935 46.99 0)
+    (property "Value" "30k 1% or NF" (id 1) (at 241.935 46.99 0)
       (effects (font (size 1.27 1.27)) (justify right))
     )
@@
     )
     (path "/0d35df78-0847-478b-9bf1-f88652133e2f"
-      (reference "R8") (unit 1) (value "10M 1% or 0R") (footprint "RevK:R_0603")
+      (reference "R8") (unit 1) (value "100k 1% or 0R") (footprint "RevK:R_0603")
     )
     (path "/00000000-0000-0000-0000-000060ce4fe8"
@@
     )
     (path "/fe9fc355-72ea-4cb8-a08f-1748e53389a5"
-      (reference "R12") (unit 1) (value "3M 1% or NF") (footprint "RevK:R_0603")
+      (reference "R12") (unit 1) (value "30k 1% or NF") (footprint "RevK:R_0603")
     )
     (path "/9edd2f4d-ab17-4d21-be4a-64fba361cb20"

Commit message: Pin names
Connections:
- net OLED-CS0 renamed OLED-CS
- net OLED-SCLK renamed OLED-SCK
- net TICK renamed GPSPPS
Changed lines of the file:
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@@
     )
   )
-  (global_label "OLED-SCLK" (shape input) (at 231.14 116.84 180) (fields_autoplaced)
+  (global_label "OLED-SCK" (shape input) (at 231.14 116.84 180) (fields_autoplaced)
     (effects (font (size 1.27 1.27)) (justify right))
-    (property "Intersheet References" "${INTERSHEET_REFS}" (id 0) (at 121.285 -13.335 0)
-      (effects (font (size 1.27 1.27)) hide)
+    (property "Intersheet References" "${INTERSHEET_REFS}" (id 0) (at 218.7163 116.7606 0)
+      (effects (font (size 1.27 1.27)) (justify right) hide)
     )
   )
@@
     )
   )
-  (global_label "OLED-CS0" (shape input) (at 231.14 119.38 180) (fields_autoplaced)
+  (global_label "OLED-CS" (shape input) (at 231.14 119.38 180) (fields_autoplaced)
     (effects (font (size 1.27 1.27)) (justify right))
-    (property "Intersheet References" "${INTERSHEET_REFS}" (id 0) (at 121.285 -13.335 0)
-      (effects (font (size 1.27 1.27)) hide)
+    (property "Intersheet References" "${INTERSHEET_REFS}" (id 0) (at 219.9863 119.3006 0)
+      (effects (font (size 1.27 1.27)) (justify right) hide)
     )
   )
@@
     )
   )
-  (global_label "OLED-CS0" (shape output) (at 81.28 83.82 0) (fields_autoplaced)
+  (global_label "OLED-CS" (shape output) (at 81.28 83.82 0) (fields_autoplaced)
     (effects (font (size 1.27 1.27)) (justify left))
-    (property "Intersheet References" "${INTERSHEET_REFS}" (id 0) (at 93.6432 83.8994 0)
+    (property "Intersheet References" "${INTERSHEET_REFS}" (id 0) (at 92.4337 83.7406 0)
       (effects (font (size 1.27 1.27)) (justify left) hide)
     )
@@
     )
   )
-  (global_label "OLED-SCLK" (shape output) (at 81.28 81.28 0) (fields_autoplaced)
+  (global_label "OLED-SCK" (shape output) (at 81.28 81.28 0) (fields_autoplaced)
     (effects (font (size 1.27 1.27)) (justify left))
-    (property "Intersheet References" "${INTERSHEET_REFS}" (id 0) (at 94.7318 81.2006 0)
+    (property "Intersheet References" "${INTERSHEET_REFS}" (id 0) (at 93.7037 81.2006 0)
       (effects (font (size 1.27 1.27)) (justify left) hide)
     )
@@
     )
   )
-  (global_label "TICK" (shape input) (at 81.28 88.9 0) (fields_autoplaced)
+  (global_label "GPSPPS" (shape input) (at 81.28 88.9 0) (fields_autoplaced)
     (effects (font (size 1.27 1.27)) (justify left))
-    (property "Intersheet References" "${INTERSHEET_REFS}" (id 0) (at 87.7166 88.9794 0)
+    (property "Intersheet References" "${INTERSHEET_REFS}" (id 0) (at 91.1032 88.8206 0)
       (effects (font (size 1.27 1.27)) (justify left) hide)
     )
@@
     )
   )
-  (global_label "TICK" (shape output) (at 78.74 139.7 0) (fields_autoplaced)
+  (global_label "GPSPPS" (shape output) (at 78.74 139.7 0) (fields_autoplaced)
     (effects (font (size 1.27 1.27)) (justify left))
-    (property "Intersheet References" "${INTERSHEET_REFS}" (id 0) (at 85.1766 139.6206 0)
+    (property "Intersheet References" "${INTERSHEET_REFS}" (id 0) (at 88.5632 139.6206 0)
       (effects (font (size 1.27 1.27)) (justify left) hide)
     )
