File: KiCad/Glider.kicad_pcb (KiCad board)
At the start: 2 copper layers, 36 x 24.5 mm, 36 parts, among them J1 DC, J2 I/O, J3 USB-C, U1 ESP32-PICO-MINI-02, U2 L96-M33, U3 FT231XQ, U4 LMR16006+FB, U5 QR

Commit message: DRC tweaks
Routing:
- net GND: track 97.6 -> 54.8 mm
- net +3V3: track 72.0 -> 71.4 mm
Other:
- rule pad_to_mask_clearance: 0 -> 0.01

Commit message: Resistors
Parts:
- R12: value 3M 1% or NF -> 30k 1% or NF
- R8: value 10M 1% or 0R -> 100k 1% or 0R
Changed lines of the file:
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@@
       (effects (font (size 0.5 0.5) (thickness 0.08)))
     )
-    (fp_text value "3M 1% or NF" (at 0 0) (layer "F.Fab")
+    (fp_text value "30k 1% or NF" (at 0 0) (layer "F.Fab")
       (effects (font (size 0.4 0.4) (thickness 0.08)))
     )
@@
       (effects (font (size 0.5 0.5) (thickness 0.08)))
     )
-    (fp_text value "10M 1% or 0R" (at 0 0 90) (layer "F.Fab")
+    (fp_text value "100k 1% or 0R" (at 0 0 90) (layer "F.Fab")
       (effects (font (size 0.4 0.4) (thickness 0.08)))
     )
