File: KiCad/Glider.kicad_sch (KiCad schematic)
At the start: 36 parts, among them J1 DC, J2 I/O, J3 USB-C, U1 ESP32-PICO-MINI-02, U2 L96-M33, U3 FT231XQ, U4 LMR16006+FB, U5 QR

Commit message: Resistors
Parts:
- R12: value 3M 1% or NF -> 30k 1% or NF
- R8: value 10M 1% or 0R -> 100k 1% or 0R
Changed lines of the file:
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@@
       (effects (font (size 1.27 1.27)) (justify left))
     )
-    (property "Value" "10M 1% or 0R" (id 1) (at 236.855 46.355 90)
+    (property "Value" "100k 1% or 0R" (id 1) (at 236.855 46.355 90)
       (effects (font (size 1.27 1.27)) (justify left))
     )
@@
       (effects (font (size 1.27 1.27)) (justify right))
     )
-    (property "Value" "3M 1% or NF" (id 1) (at 241.935 46.99 0)
+    (property "Value" "30k 1% or NF" (id 1) (at 241.935 46.99 0)
       (effects (font (size 1.27 1.27)) (justify right))
     )
@@
     )
     (path "/0d35df78-0847-478b-9bf1-f88652133e2f"
-      (reference "R8") (unit 1) (value "10M 1% or 0R") (footprint "RevK:R_0603")
+      (reference "R8") (unit 1) (value "100k 1% or 0R") (footprint "RevK:R_0603")
     )
     (path "/00000000-0000-0000-0000-000060ce4fe8"
@@
     )
     (path "/fe9fc355-72ea-4cb8-a08f-1748e53389a5"
-      (reference "R12") (unit 1) (value "3M 1% or NF") (footprint "RevK:R_0603")
+      (reference "R12") (unit 1) (value "30k 1% or NF") (footprint "RevK:R_0603")
     )
     (path "/a68666c5-d248-40dd-b132-5bb6a20a9cf7"
