File: PCB/L86/L86.kicad_pcb (KiCad board)
At the start: 2 copper layers, 38.5 x 30 mm, 4 parts, among them J1 Conn_01x06, U1 L86-M33, U2 QR

Commit message: Moved from SS
Parts:
- removed U2: QR, RevK:QR-GPS
- added BT1: Battery_Cell, RevK:Battery-Holder-2032, B.Cu at (100.0, 97.0)
- added Logo2: AJK, RevK:AJK, B.Cu at (114.0, 112.0)
- J1: value Conn_01x06 -> Conn_01x05; footprint RevK:Molex_MiniSPOX_H6RA -> RevK:PTSM-HH-5-RA-P-SMD; moved to B.Cu
- Logo1: value AJK -> AA; footprint RevK:AJK -> RevK:AA
- moved J1 19.6 mm to (100.0, 109.9), turned to 180 degrees
- moved Logo1 14.6 mm to (112.0, 88.0), turned to 90 degrees
- turned U1 to -90 degrees
Connections:
- J1 pad 1: Net-(J1-Pad1) -> GND
- J1 pad 2: Net-(J1-Pad2) -> Net-(J1-Pin_2)
- J1 pad 3: GND -> Net-(J1-Pin_3)
- J1 pad 4: Net-(J1-Pad4) -> Net-(J1-Pin_4)
- J1 pad 5: Net-(J1-Pad5) -> Net-(J1-Pin_5)
- U1 pad 1: Net-(J1-Pad1) -> Net-(J1-Pin_2)
- U1 pad 12: unconnected-(U1-Pad12) -> GND
- U1 pad 2: Net-(J1-Pad2) -> Net-(J1-Pin_3)
- U1 pad 4: Net-(J1-Pad4) -> Net-(J1-Pin_5)
- U1 pad 5: Net-(J1-Pad5) -> BAT
- U1 pad 6: Net-(J1-Pad6) -> Net-(J1-Pin_4)
Routing:
- net BAT: track 0.00 -> 15.0 mm, vias 0 -> 1
- net Net-(J1-Pad1): track 13.0 -> 0.00 mm, vias 1 -> 0
- net Net-(J1-Pad2): track 13.0 -> 0.00 mm, vias 1 -> 0
- net Net-(J1-Pad4): track 12.9 -> 0.00 mm, vias 1 -> 0
- net Net-(J1-Pad5): track 12.9 -> 0.00 mm, vias 1 -> 0
- net Net-(J1-Pad6): track 12.9 -> 0.00 mm, vias 1 -> 0
- net Net-(J1-Pin_5): track 0.00 -> 12.1 mm, vias 0 -> 1
- net Net-(J1-Pin_3): track 0.00 -> 8.03 mm, vias 0 -> 1
- net Net-(J1-Pin_2): track 0.00 -> 6.77 mm, vias 0 -> 1
- net Net-(J1-Pin_4): track 0.00 -> 4.97 mm, vias 0 -> 1
- net GND: vias 0 -> 1
Other:
- board size 38.5 x 30 mm -> 36 x 36 mm
- rule pad_to_mask_clearance: 0.01 -> 0
- board text added: "${CURRENT_DATE}"
- board text added: "+"
- board text added: "<"
- board text added: ">"
- board text added: "GPS"
- board text added: "⎍"
- board text added: "⏚"
- board text removed: "BAT"
- board text removed: "GND"
- board text removed: "PPS"
- board text removed: "VCC"
- board text removed: "←TX"
- board text removed: "→RX"

Commit message: SS
Parts:
- moved Logo1 34.7 mm to (87.0, 112.0)
Other:
- board text added: "CR2032"

Commit message: Cap
Parts:
- added C1: C_Polarized, RevK:CP_EIA-7343-31_Kemet-D, B.Cu at (113.0, 105.0)
Routing:
- net Net-(J1-Pin_5): track 12.1 -> 19.1 mm

Commit message: ESD
Parts:
- added D1: ~, RevK:DFN1006-2L, B.Cu at (98.8, 109.0)
- added D2: ~, RevK:DFN1006-2L, B.Cu at (101.2, 109.0)
- added D3: ~, RevK:DFN1006-2L, B.Cu at (96.2, 109.0)
- added D4: ~, RevK:DFN1006-2L, B.Cu at (103.8, 109.0)
Routing:
- net GND: track 0.00 -> 12.3 mm
- net Net-(J1-Pin_4): track 4.97 -> 7.55 mm
- net Net-(J1-Pin_5): track 19.1 -> 21.1 mm
- net Net-(J1-Pin_3): track 8.03 -> 9.83 mm
- net Net-(J1-Pin_2): track 6.77 -> 8.16 mm
- net BAT: track 15.0 -> 13.8 mm

Commit message: EAN
Other:
- board text added: "5060634238177"

Commit message: Tweak
Other:
- board text added: "C"
- board text added: "M"
