File: PCB/L86/L86.kicad_pcb (KiCad board)
At the start: 2 copper layers, 36 x 36 mm, 10 parts, among them J1 Conn_01x05, U1 L86-M33

Commit message: Position adjust
Routing:
- net Net-(J1-Pin_3): track 9.83 -> 10.8 mm
- net Net-(J1-Pin_5): track 21.1 -> 20.4 mm
