File: PCB/L86/L86.kicad_sch (KiCad schematic)
At the start: 4 parts, among them J1 Conn_01x06, U1 L86-M33, U2 QR

Commit message: Moved from SS
Parts:
- removed J1: Conn_01x06, RevK:Molex_MiniSPOX_H6RA, symbol Connector_Generic:Conn_01x06
- removed Logo1: AJK, RevK:AJK, symbol RevK:AJK
- removed U2: QR, RevK:QR-GPS, symbol RevK:QR
- added BT1: Battery_Cell, RevK:Battery-Holder-2032, symbol Device:Battery_Cell
- added J1: Conn_01x05, RevK:PTSM-HH-5-RA-P-SMD, symbol Connector_Generic:Conn_01x05
- added Logo1: AA, RevK:AA, symbol RevK:AA
- added Logo2: AJK, RevK:AJK, symbol RevK:AJK
Connections:
- net GND: now also U1.12 (GND), BT1.2 (-), J1.1 (Pin_1)
- net at U1.1 (RXD1): now also J1.2 (Pin_2)
- net at U1.2 (TXD1): now also J1.3 (Pin_3)
- net at U1.4 (VCC): now also J1.5 (Pin_5)
- net BAT: now reaches U1.5 (V_BKCP)
- net BAT: now also BT1.1 (+)
- net at U1.6 (1PPS): now also J1.4 (Pin_4)
- no-connect marks 5 -> 4
Other:
- company: (none) -> Adrian Kennard Andrews & Arnold Ltd
- title: (none) -> GPS reference

Commit message: Cap
Parts:
- added C28: C_Polarized, RevK:CP_EIA-7343-31_Kemet-D, symbol Device:C_Polarized
Connections:
- net GND: now also C28.2
- net at J1.5 (Pin_5), U1.4 (VCC): now also C28.1
Other:
- moved on the sheet: J1
Changed lines of the file:
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@@
     (comment 2 "www.me.uk")
+  )
+  (junction (at 129.54 72.39) (diameter 0) (color 0 0 0 0)
   )
   (junction (at 121.92 82.55) (diameter 0) (color 0 0 0 0)
@@
     (stroke (width 0) (type default))
   )
+  (wire (pts (xy 116.84 80.01) (xy 148.59 80.01))
+    (stroke (width 0) (type default))
+  )
+  (wire (pts (xy 116.84 67.31) (xy 124.46 67.31))
+    (stroke (width 0) (type default))
+  )
+  (wire (pts (xy 124.46 67.31) (xy 124.46 74.93))
+    (stroke (width 0) (type default))
+  )
+  (wire (pts (xy 121.92 82.55) (xy 121.92 85.09))
+    (stroke (width 0) (type default))
+  )
+  (wire (pts (xy 116.84 72.39) (xy 129.54 72.39))
+    (stroke (width 0) (type default))
+  )
+  (wire (pts (xy 129.54 72.39) (xy 148.59 72.39))
+    (stroke (width 0) (type default))
+  )
   (wire (pts (xy 121.92 74.93) (xy 121.92 82.55))
     (stroke (width 0) (type default))
   )
-  (wire (pts (xy 116.84 67.31) (xy 124.46 67.31))
-    (stroke (width 0) (type default))
-  )
-  (wire (pts (xy 116.84 80.01) (xy 128.27 80.01))
-    (stroke (width 0) (type default))
-  )
-  (wire (pts (xy 124.46 67.31) (xy 124.46 74.93))
-    (stroke (width 0) (type default))
-  )
-  (wire (pts (xy 116.84 77.47) (xy 128.27 77.47))
-    (stroke (width 0) (type default))
-  )
-  (wire (pts (xy 116.84 72.39) (xy 128.27 72.39))
-    (stroke (width 0) (type default))
-  )
-  (wire (pts (xy 121.92 82.55) (xy 121.92 85.09))
-    (stroke (width 0) (type default))
-  )
-  (wire (pts (xy 121.92 82.55) (xy 128.27 82.55))
-    (stroke (width 0) (type default))
-  )
-  (wire (pts (xy 124.46 74.93) (xy 128.27 74.93))
+  (wire (pts (xy 121.92 82.55) (xy 148.59 82.55))
+    (stroke (width 0) (type default))
+  )
+  (wire (pts (xy 124.46 74.93) (xy 148.59 74.93))
+    (stroke (width 0) (type default))
+  )
+  (wire (pts (xy 116.84 77.47) (xy 148.59 77.47))
     (stroke (width 0) (type default))
   )
@@
     )
   )
-  (symbol (lib_id "Connector_Generic:Conn_01x05") (at 133.35 77.47 0) (mirror x) (unit 1)
-    (in_bom yes) (on_board yes) (dnp no) (fields_autoplaced)
-    (property "Reference" "J1" (at 133.35 67.4202 0)
-      (effects (font (size 1.27 1.27)))
-    )
-    (property "Value" "Conn_01x05" (at 133.35 69.9571 0)
-      (effects (font (size 1.27 1.27)))
-    )
-    (property "Footprint" "RevK:PTSM-HH-5-RA-P-SMD" (at 133.35 77.47 0)
-      (effects (font (size 1.27 1.27)) hide)
-    )
-    (property "Datasheet" "~" (at 133.35 77.47 0)
-      (effects (font (size 1.27 1.27)) hide)
-    )
-    (property "Phenoix part" "1814948" (at 133.35 77.47 0)
+  (symbol (lib_id "Connector_Generic:Conn_01x05") (at 153.67 77.47 0) (mirror x) (unit 1)
+    (in_bom yes) (on_board yes) (dnp no) (fields_autoplaced)
+    (property "Reference" "J1" (at 153.67 67.4202 0)
+      (effects (font (size 1.27 1.27)))
+    )
+    (property "Value" "Conn_01x05" (at 153.67 69.9571 0)
+      (effects (font (size 1.27 1.27)))
+    )
+    (property "Footprint" "RevK:PTSM-HH-5-RA-P-SMD" (at 153.67 77.47 0)
+      (effects (font (size 1.27 1.27)) hide)
+    )
+    (property "Datasheet" "~" (at 153.67 77.47 0)
+      (effects (font (size 1.27 1.27)) hide)
+    )
+    (property "Phenoix part" "1814948" (at 153.67 77.47 0)
       (effects (font (size 1.27 1.27)) hide)
     )
@@
         (path "/babeabf2-f3b0-4ed5-8d9e-0215947e6cf3"
           (reference "J1") (unit 1)
+        )
+      )
+    )
+  )
+  (symbol (lib_name "GND_1") (lib_id "power:GND") (at 129.54 64.77 180) (unit 1)
+    (in_bom yes) (on_board yes) (dnp no) (fields_autoplaced)
+    (property "Reference" "#PWR01" (at 129.54 58.42 0)
+      (effects (font (size 1.27 1.27)) hide)
+    )
+    (property "Value" "GND" (at 129.54 60.6369 0)
+      (effects (font (size 1.27 1.27)))
+    )
+    (property "Footprint" "" (at 129.54 64.77 0)
+      (effects (font (size 1.27 1.27)) hide)
+    )
+    (property "Datasheet" "" (at 129.54 64.77 0)
+      (effects (font (size 1.27 1.27)) hide)
+    )
+    (pin "1")
+    (instances
+      (project "L86"
+        (path "/babeabf2-f3b0-4ed5-8d9e-0215947e6cf3"
+          (reference "#PWR01") (unit 1)
         )
       )
@@
         )
       )
+    )
+  )
+  (symbol (lib_id "Device:C_Polarized") (at 129.54 68.58 180) (unit 1)
+    (in_bom yes) (on_board yes) (dnp no) (fields_autoplaced)
+    (property "Reference" "C28" (at 132.461 68.2569 0)
+      (effects (font (size 1.27 1.27)) (justify right))
+    )
+    (property "Value" "C_Polarized" (at 132.461 70.6811 0)
+      (effects (font (size 1.27 1.27)) (justify right))
+    )
+    (property "Footprint" "RevK:CP_EIA-7343-31_Kemet-D" (at 128.5748 64.77 0)
+      (effects (font (size 1.27 1.27)) hide)
+    )
+    (property "Datasheet" "~" (at 129.54 68.58 0)
+      (effects (font (size 1.27 1.27)) hide)
+    )
+    (property "LCSC Part #" "C106188" (at 129.54 68.58 0)
+      (effects (font (size 1.27 1.27)) hide)
+    )
+    (property "JLCPCB Rotation Offset" "180" (at 129.54 68.58 0)
+      (effects (font (size 1.27 1.27)) hide)
+    )
+    (pin "1")
+    (pin "2")
+    (instances
+      (project "EPD75"
+        (path "/46c350bb-7de4-4e81-aafd-4af55e37aab0"
+          (reference "C28") (unit 1)
+        )
+      )
+      (project "L86"
+        (path "/babeabf2-f3b0-4ed5-8d9e-0215947e6cf3"
+          (reference "C1") (unit 1)
+        )
+      )

Commit message: ESD
Parts:
- added D27 (x4): ~, RevK:DFN1006-2L, symbol RevK:ES05D1MC10
Connections:
- net GND: now also D27.2, D27.2, D27.2, D27.2
- net at J1.2 (Pin_2), U1.1 (RXD1): now also D27.1
- net at J1.3 (Pin_3), U1.2 (TXD1): now also D27.1
- net at J1.4 (Pin_4), U1.6 (1PPS): now also D27.1
- net at C28.1, J1.5 (Pin_5), U1.4 (VCC): now also D27.1

Commit message: Tidy
Parts:
- J1: symbol Connector_Generic:Conn_01x05 -> Connector_Generic:Conn_01x07; Part name (none) -> PTSM 0,5/ 5-HHI0-2,5SMDWH; Phenoix part 1814948 -> 1815222
Connections:
- net GND: now also J1.6 (Pin_6), J1.7 (Pin_7)
Changed lines of the file:
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@@
   (junction (at 147.32 72.39) (diameter 0) (color 0 0 0 0)
+  )
+  (junction (at 148.59 67.31) (diameter 0) (color 0 0 0 0)
   )
   (junction (at 121.92 82.55) (diameter 0) (color 0 0 0 0)
@@
     (stroke (width 0) (type default))
   )
+  (wire (pts (xy 148.59 67.31) (xy 148.59 69.85))
+    (stroke (width 0) (type default))
+  )
   (wire (pts (xy 116.84 77.47) (xy 139.7 77.47))
     (stroke (width 0) (type default))
@@
     )
   )
-  (symbol (lib_id "Connector_Generic:Conn_01x05") (at 153.67 77.47 0) (mirror x) (unit 1)
-    (in_bom yes) (on_board yes) (dnp no) (fields_autoplaced)
-    (property "Reference" "J1" (at 153.67 67.4202 0)
-      (effects (font (size 1.27 1.27)))
-    )
-    (property "Value" "Conn_01x05" (at 153.67 69.9571 0)
-      (effects (font (size 1.27 1.27)))
-    )
-    (property "Footprint" "RevK:PTSM-HH-5-RA-P-SMD" (at 153.67 77.47 0)
-      (effects (font (size 1.27 1.27)) hide)
-    )
-    (property "Datasheet" "~" (at 153.67 77.47 0)
-      (effects (font (size 1.27 1.27)) hide)
-    )
-    (property "Phenoix part" "1814948" (at 153.67 77.47 0)
+  (symbol (lib_name "GND_1") (lib_id "power:GND") (at 148.59 67.31 270) (unit 1)
+    (in_bom yes) (on_board yes) (dnp no) (fields_autoplaced)
+    (property "Reference" "#PWR08" (at 142.24 67.31 0)
+      (effects (font (size 1.27 1.27)) hide)
+    )
+    (property "Value" "GND" (at 145.4151 67.31 90)
+      (effects (font (size 1.27 1.27)) (justify right))
+    )
+    (property "Footprint" "" (at 148.59 67.31 0)
+      (effects (font (size 1.27 1.27)) hide)
+    )
+    (property "Datasheet" "" (at 148.59 67.31 0)
+      (effects (font (size 1.27 1.27)) hide)
+    )
+    (pin "1")
+    (instances
+      (project "L86"
+        (path "/babeabf2-f3b0-4ed5-8d9e-0215947e6cf3"
+          (reference "#PWR08") (unit 1)
+        )
+      )
+    )
+  )
+  (symbol (lib_id "Connector_Generic:Conn_01x07") (at 153.67 74.93 0) (mirror x) (unit 1)
+    (in_bom yes) (on_board yes) (dnp no) (fields_autoplaced)
+    (property "Reference" "J1" (at 153.67 61.8957 0)
+      (effects (font (size 1.27 1.27)))
+    )
+    (property "Value" "Conn_01x05" (at 153.67 64.3199 0)
+      (effects (font (size 1.27 1.27)))
+    )
+    (property "Footprint" "RevK:PTSM-HH-5-RA-P-SMD" (at 153.67 74.93 0)
+      (effects (font (size 1.27 1.27)) hide)
+    )
+    (property "Datasheet" "~" (at 153.67 74.93 0)
+      (effects (font (size 1.27 1.27)) hide)
+    )
+    (property "Phenoix part" "1815222" (at 153.67 74.93 0)
+      (effects (font (size 1.27 1.27)) hide)
+    )
+    (property "Part name" "PTSM 0,5/ 5-HHI0-2,5SMDWH" (at 153.67 74.93 0)
       (effects (font (size 1.27 1.27)) hide)
     )
@@
     (pin "4")
     (pin "5")
-    (instances
-      (project "L86"
+    (pin "6")
+    (pin "7")
+    (instances
+      (project "L86"

Commit message: PCB Update
Parts:
- C1: renamed from C28; JLCPCB Rotation Offset 180 -> (none); LCSC Part # C106188 -> (none); MPN (none) -> C106188
- D1, D2, D3, D4: renamed from D27; LCSC Part # C5137770 -> (none); MPN (none) -> C5137770
