File: PCB/Logger/Logger.kicad_sch (KiCad schematic)
At the start: 74 parts, among them J2 USB-C-Socket-V, J3 JST-PH-SM4-TB, J3 USB-PROG, J5 Conn_01x05, J6 TF_PUSH, J8 Shelly, Q1 C179347, Q4 CJ2301, U1 TP4054, U10 ESP32-S3-MINI-1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

Commit message: Tweak
Connections:
- net ADC renamed ADC1
Other:
- moved on the sheet: R12, R13
Changed lines of the file:
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@@
   (junction (at 124.46 154.305) (diameter 0) (color 0 0 0 0)
   )
-  (junction (at 247.65 37.465) (diameter 0) (color 0 0 0 0)
+  (junction (at 252.73 144.78) (diameter 0) (color 0 0 0 0)
   )
   (junction (at 173.355 29.845) (diameter 0) (color 0 0 0 0)
@@
   (no_connect (at 42.545 48.26))
   (no_connect (at 73.025 66.04))
-  (no_connect (at 213.995 119.38))
   (no_connect (at 201.295 106.045))
+  (no_connect (at 213.995 119.38))
   (no_connect (at 73.025 60.96))
   (no_connect (at 73.025 81.28))
@@
     (stroke (width 0) (type default))
   )
-  (wire (pts (xy 251.46 37.465) (xy 247.65 37.465))
+  (wire (pts (xy 256.54 144.78) (xy 252.73 144.78))
     (stroke (width 0) (type default))
   )
@@
     )
   )
-  (global_label "ADC" (shape output) (at 251.46 37.465 0)
+  (global_label "ADC1" (shape output) (at 256.54 144.78 0)
     (effects (font (size 1.27 1.27)) (justify left))
-    (property "Intersheetrefs" "${INTERSHEET_REFS}" (at 251.46 37.465 0)
+    (property "Intersheetrefs" "${INTERSHEET_REFS}" (at 256.54 144.78 0)
       (effects (font (size 1.27 1.27)) hide)
     )
@@
     )
   )
-  (global_label "ADC" (shape input) (at 198.12 106.045 90)
+  (global_label "ADC1" (shape input) (at 198.12 106.045 90)
     (effects (font (size 1.27 1.27)) (justify left))
     (property "Intersheetrefs" "${INTERSHEET_REFS}" (at 198.12 106.045 0)
@@
     )
   )
-  (global_label "VBAT" (shape input) (at 247.65 22.225 90) (fields_autoplaced)
+  (global_label "VBAT" (shape input) (at 252.73 129.54 90) (fields_autoplaced)
     (effects (font (size 1.27 1.27)) (justify left))
-    (property "Intersheetrefs" "${INTERSHEET_REFS}" (at 247.65 15.4792 90)
+    (property "Intersheetrefs" "${INTERSHEET_REFS}" (at 252.73 122.7942 90)
       (effects (font (size 1.27 1.27)) (justify left) hide)
     )
@@
     )
   )
-  (symbol (lib_id "Device:R") (at 247.65 41.275 0) (unit 1)
+  (symbol (lib_id "Device:R") (at 252.73 148.59 0) (unit 1)
     (in_bom yes) (on_board yes) (dnp no)
-    (property "Reference" "R13" (at 247.65 41.275 90)
+    (property "Reference" "R13" (at 252.73 148.59 90)
       (effects (font (size 1.27 1.27)))
     )
-    (property "Value" "100K 1%" (at 250.19 43.18 90)
+    (property "Value" "100K 1%" (at 255.27 150.495 90)
       (effects (font (size 1.27 1.27)))
     )
-    (property "Footprint" "RevK:R_0402" (at 245.872 41.275 90)
+    (property "Footprint" "RevK:R_0402" (at 250.952 148.59 90)
       (effects (font (size 1.27 1.27)) hide)
     )
-    (property "Datasheet" "~" (at 247.65 41.275 0)
+    (property "Datasheet" "~" (at 252.73 148.59 0)
       (effects (font (size 1.27 1.27)) hide)
     )
-    (property "LCSC Part #" "C5139597" (at 247.65 41.275 90)
+    (property "LCSC Part #" "C5139597" (at 252.73 148.59 90)
       (effects (font (size 1.27 1.27)) hide)
     )
@@
     )
   )
-  (symbol (lib_id "power:GND") (at 247.65 45.085 0) (unit 1)
+  (symbol (lib_id "power:GND") (at 252.73 152.4 0) (unit 1)
     (in_bom yes) (on_board yes) (dnp no)
-    (property "Reference" "#PWR046" (at 247.65 51.435 0)
+    (property "Reference" "#PWR046" (at 252.73 158.75 0)
       (effects (font (size 1.27 1.27)) hide)
     )
-    (property "Value" "GND" (at 247.65 48.895 0)
+    (property "Value" "GND" (at 252.73 156.21 0)
       (effects (font (size 1.27 1.27)))
     )
-    (property "Footprint" "" (at 247.65 45.085 0)
+    (property "Footprint" "" (at 252.73 152.4 0)
       (effects (font (size 1.27 1.27)) hide)
     )
-    (property "Datasheet" "" (at 247.65 45.085 0)
+    (property "Datasheet" "" (at 252.73 152.4 0)
       (effects (font (size 1.27 1.27)) hide)
     )
@@
     )
   )
-  (symbol (lib_id "Device:R") (at 247.65 33.655 0) (unit 1)
+  (symbol (lib_id "Device:R") (at 252.73 140.97 0) (unit 1)
     (in_bom yes) (on_board yes) (dnp no)
-    (property "Reference" "R12" (at 247.65 33.655 90)
+    (property "Reference" "R12" (at 252.73 140.97 90)
       (effects (font (size 1.27 1.27)))
     )
-    (property "Value" "100K 1%" (at 245.11 33.02 90)
+    (property "Value" "100K 1%" (at 250.19 140.335 90)
       (effects (font (size 1.27 1.27)))
     )
-    (property "Footprint" "RevK:R_0402" (at 245.872 33.655 90)
+    (property "Footprint" "RevK:R_0402" (at 250.952 140.97 90)
       (effects (font (size 1.27 1.27)) hide)
     )
-    (property "Datasheet" "~" (at 247.65 33.655 0)
+    (property "Datasheet" "~" (at 252.73 140.97 0)
       (effects (font (size 1.27 1.27)) hide)
     )
-    (property "LCSC Part #" "C5139597" (at 247.65 33.655 90)
+    (property "LCSC Part #" "C5139597" (at 252.73 140.97 90)
       (effects (font (size 1.27 1.27)) hide)
     )
@@
     )
   )
-  (symbol (lib_id "Device:R") (at 247.65 26.035 0) (unit 1)
+  (symbol (lib_id "Device:R") (at 252.73 133.35 0) (unit 1)
     (in_bom yes) (on_board yes) (dnp no)
-    (property "Reference" "R12" (at 247.65 26.035 90)
+    (property "Reference" "R12" (at 252.73 133.35 90)
       (effects (font (size 1.27 1.27)))
     )
-    (property "Value" "100K 1%" (at 250.19 25.4 90)
+    (property "Value" "100K 1%" (at 255.27 132.715 90)
       (effects (font (size 1.27 1.27)))
     )
-    (property "Footprint" "RevK:R_0402" (at 245.872 26.035 90)
+    (property "Footprint" "RevK:R_0402" (at 250.952 133.35 90)
       (effects (font (size 1.27 1.27)) hide)
     )
-    (property "Datasheet" "~" (at 247.65 26.035 0)
+    (property "Datasheet" "~" (at 252.73 133.35 0)
       (effects (font (size 1.27 1.27)) hide)
     )
-    (property "LCSC Part #" "C5139597" (at 247.65 26.035 90)
+    (property "LCSC Part #" "C5139597" (at 252.73 133.35 90)
       (effects (font (size 1.27 1.27)) hide)
     )

Commit message: Rework
Parts:
- added R10: 1R 1W, RevK:R_1218, symbol Device:R
Connections:
- net +3.3V: now also R10.2; no longer Q1.2 (S), R1.1
- new net: Q1.2 (S), R1.1, R10.1
Other:
- moved on the sheet: C28
Changed lines of the file:
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@@
   (junction (at 167.64 161.925) (diameter 0) (color 0 0 0 0)
   )
+  (junction (at 163.195 71.755) (diameter 0) (color 0 0 0 0)
+  )
   (junction (at 71.12 120.65) (diameter 0) (color 0 0 0 0)
   )
@@
   (junction (at 70.485 161.925) (diameter 0) (color 0 0 0 0)
   )
-  (junction (at 155.575 71.755) (diameter 0) (color 0 0 0 0)
-  )
   (junction (at 97.79 154.305) (diameter 0) (color 0 0 0 0)
   )
@@
   (junction (at 178.435 154.305) (diameter 0) (color 0 0 0 0)
   )
-  (junction (at 163.195 71.755) (diameter 0) (color 0 0 0 0)
-  )
   (junction (at 119.38 161.925) (diameter 0) (color 0 0 0 0)
   )
@@
     (stroke (width 0) (type default))
   )
+  (wire (pts (xy 163.195 70.485) (xy 163.195 71.755))
+    (stroke (width 0) (type default))
+  )
   (wire (pts (xy 123.19 60.325) (xy 127.635 60.325))
     (stroke (width 0) (type default))
@@
     (stroke (width 0) (type default))
   )
-  (wire (pts (xy 155.575 66.04) (xy 155.575 71.755))
-    (stroke (width 0) (type default))
-  )
   (wire (pts (xy 151.765 161.925) (xy 156.845 161.925))
     (stroke (width 0) (type default))
@@
     )
   )
+  (symbol (lib_id "Device:R") (at 163.195 66.675 180) (unit 1)
+    (in_bom yes) (on_board yes) (dnp no)
+    (property "Reference" "R10" (at 163.195 67.31 90)
+      (effects (font (size 1.27 1.27)))
+    )
+    (property "Value" "1R 1W" (at 160.4589 66.675 90)
+      (effects (font (size 1.27 1.27)))
+    )
+    (property "Footprint" "RevK:R_1218" (at 164.973 66.675 90)
+      (effects (font (size 1.27 1.27)) hide)
+    )
+    (property "Datasheet" "~" (at 163.195 66.675 0)
+      (effects (font (size 1.27 1.27)) hide)
+    )
+    (property "LCSC Part #" "C175540" (at 163.195 66.675 0)
+      (effects (font (size 1.27 1.27)) hide)
+    )
+    (pin "2")
+    (pin "1")
+    (instances
+      (project "Logger"
+        (path "/babeabf2-f3b0-4ed5-8d9e-0215947e6cf3"
+          (reference "R10") (unit 1)
+        )
+      )
+    )
+  )
   (symbol (lib_id "power:GND") (at 185.42 124.46 270) (unit 1)
     (in_bom yes) (on_board yes) (dnp no) (fields_autoplaced)
@@
     )
   )
-  (symbol (lib_id "Device:C_Polarized") (at 155.575 62.23 180) (unit 1)
-    (in_bom yes) (on_board yes) (dnp no) (fields_autoplaced)
-    (property "Reference" "C28" (at 158.496 61.9069 0)
+  (symbol (lib_id "Device:C_Polarized") (at 57.15 20.32 270) (unit 1)
+    (in_bom yes) (on_board yes) (dnp no)
+    (property "Reference" "C28" (at 55.245 18.415 90)
       (effects (font (size 1.27 1.27)) (justify right))
     )
-    (property "Value" "C_Polarized" (at 158.496 64.3311 0)
+    (property "Value" "C_Polarized" (at 62.23 24.13 90)
       (effects (font (size 1.27 1.27)) (justify right))
     )
-    (property "Footprint" "RevK:CP_EIA-7343-31_Kemet-D" (at 154.6098 58.42 0)
+    (property "Footprint" "RevK:CP_EIA-7343-31_Kemet-D" (at 53.34 21.2852 0)
       (effects (font (size 1.27 1.27)) hide)
     )
-    (property "Datasheet" "~" (at 155.575 62.23 0)
+    (property "Datasheet" "~" (at 57.15 20.32 0)
       (effects (font (size 1.27 1.27)) hide)
     )
-    (property "LCSC Part #" "C106188" (at 155.575 62.23 0)
+    (property "LCSC Part #" "C106188" (at 57.15 20.32 0)
       (effects (font (size 1.27 1.27)) hide)
     )
-    (property "JLCPCB Rotation Offset" "180" (at 155.575 62.23 0)
+    (property "JLCPCB Rotation Offset" "180" (at 57.15 20.32 0)
       (effects (font (size 1.27 1.27)) hide)
     )
@@
     )
   )
+  (symbol (lib_id "power:+3.3V") (at 60.96 20.32 270) (unit 1)
+    (in_bom yes) (on_board yes) (dnp no) (fields_autoplaced)
+    (property "Reference" "#PWR060" (at 57.15 20.32 0)
+      (effects (font (size 1.27 1.27)) hide)
+    )
+    (property "Value" "+3.3V" (at 65.0931 20.32 0)
+      (effects (font (size 1.27 1.27)))
+    )
+    (property "Footprint" "" (at 60.96 20.32 0)
+      (effects (font (size 1.27 1.27)) hide)
+    )
+    (property "Datasheet" "" (at 60.96 20.32 0)
+      (effects (font (size 1.27 1.27)) hide)
+    )
+    (pin "1")
+    (instances
+      (project "Access"
+        (path "/2a267270-6585-45e3-a633-b53049f10066"
+          (reference "#PWR060") (unit 1)
+        )
+      )
+      (project "USBA"
+        (path "/2d210a96-f81f-42a9-8bf4-1b43c11086f3"
+          (reference "#PWR03") (unit 1)
+        )
+      )
+      (project "Faikin"
+        (path "/46c350bb-7de4-4e81-aafd-4af55e37aab0"
+          (reference "#PWR012") (unit 1)
+        )
+      )
+      (project "Bell"
+        (path "/770ad51a-7219-4633-b24a-bd20feb0a6c5"
+          (reference "#PWR032") (unit 1)
+        )
+      )
+      (project "Logger"
+        (path "/babeabf2-f3b0-4ed5-8d9e-0215947e6cf3"
+          (reference "#PWR042") (unit 1)
+        )
+      )
+    )
+  )
   (symbol (lib_id "RevK:WS2812B-1mm") (at 178.435 158.115 0) (mirror x) (unit 1)
     (in_bom yes) (on_board yes) (dnp no)
@@
     )
   )
-  (symbol (lib_id "power:+3.3V") (at 163.195 71.755 0) (unit 1)
+  (symbol (lib_id "power:+3.3V") (at 163.195 62.865 0) (unit 1)
     (in_bom yes) (on_board yes) (dnp no) (fields_autoplaced)
-    (property "Reference" "#PWR021" (at 163.195 75.565 0)
+    (property "Reference" "#PWR021" (at 163.195 66.675 0)
       (effects (font (size 1.27 1.27)) hide)
     )
-    (property "Value" "+3.3V" (at 163.195 67.6219 0)
-      (effects (font (size 1.27 1.27)))
+    (property "Value" "+3.3V" (at 163.195 59.69 90)
+      (effects (font (size 1.27 1.27)) (justify left))
     )
-    (property "Footprint" "" (at 163.195 71.755 0)
+    (property "Footprint" "" (at 163.195 62.865 0)
       (effects (font (size 1.27 1.27)) hide)
     )
-    (property "Datasheet" "" (at 163.195 71.755 0)
+    (property "Datasheet" "" (at 163.195 62.865 0)
       (effects (font (size 1.27 1.27)) hide)
     )
@@
     )
   )
-  (symbol (lib_id "power:GND") (at 155.575 58.42 180) (unit 1)
+  (symbol (lib_id "power:GND") (at 53.34 20.32 270) (unit 1)
     (in_bom yes) (on_board yes) (dnp no) (fields_autoplaced)
-    (property "Reference" "#PWR0105" (at 155.575 52.07 0)
+    (property "Reference" "#PWR0105" (at 46.99 20.32 0)
       (effects (font (size 1.27 1.27)) hide)
     )
-    (property "Value" "GND" (at 155.575 54.2869 0)
+    (property "Value" "GND" (at 49.2069 20.32 0)
       (effects (font (size 1.27 1.27)))
     )
-    (property "Footprint" "" (at 155.575 58.42 0)
+    (property "Footprint" "" (at 53.34 20.32 0)
       (effects (font (size 1.27 1.27)) hide)
     )
-    (property "Datasheet" "" (at 155.575 58.42 0)
+    (property "Datasheet" "" (at 53.34 20.32 0)
       (effects (font (size 1.27 1.27)) hide)
     )

Commit message: Tidy
Parts:
- added Q4: CJ2301, RevK:SOT-23, symbol Transistor_FET:BSS83P
- added R12: 100K 1%, RevK:R_0402, symbol Device:R
Connections:
- net +3.3V: now also Q4.3 (D)
- net GND: now also R12.2
- net VBUS: now also Q4.1 (G), R12.1
- net USB: now reaches U10.10 (GPIO6)
- net USB: now also Q4.2 (S)
- net CHARGER renamed CHARGING
- no-connect marks 26 -> 25
Changed lines of the file:
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@@
   (junction (at 179.705 32.385) (diameter 0) (color 0 0 0 0)
   )
+  (junction (at 222.25 40.005) (diameter 0) (color 0 0 0 0)
+  )
   (junction (at 86.995 154.305) (diameter 0) (color 0 0 0 0)
   )
@@
   (no_connect (at 73.025 71.12))
   (no_connect (at 42.545 86.36))
-  (no_connect (at 42.545 48.26))
   (no_connect (at 73.025 66.04))
   (no_connect (at 201.295 106.045))
@@
     (stroke (width 0) (type default))
   )
+  (wire (pts (xy 219.71 40.005) (xy 222.25 40.005))
+    (stroke (width 0) (type default))
+  )
   (wire (pts (xy 130.81 60.325) (xy 130.81 65.405))
     (stroke (width 0) (type default))
@@
     (stroke (width 0) (type default))
   )
+  (wire (pts (xy 229.87 45.085) (xy 229.87 47.625))
+    (stroke (width 0) (type default))
+  )
   (wire (pts (xy 163.195 70.485) (xy 163.195 71.755))
     (stroke (width 0) (type default))
@@
     (stroke (width 0) (type default))
   )
-  (global_label "CHARGER" (shape input) (at 42.545 43.18 180) (fields_autoplaced)
+  (global_label "CHARGING" (shape input) (at 42.545 43.18 180) (fields_autoplaced)
     (effects (font (size 1.27 1.27)) (justify right))
-    (property "Intersheetrefs" "${INTERSHEET_REFS}" (at 31.5659 43.18 0)
+    (property "Intersheetrefs" "${INTERSHEET_REFS}" (at 30.7796 43.18 0)
       (effects (font (size 1.27 1.27)) (justify right) hide)
     )
@@
     )
   )
-  (global_label "CHARGER" (shape output) (at 137.795 37.465 0) (fields_autoplaced)
+  (global_label "CHARGING" (shape output) (at 137.795 37.465 0) (fields_autoplaced)
     (effects (font (size 1.27 1.27)) (justify left))
-    (property "Intersheetrefs" "${INTERSHEET_REFS}" (at 148.7741 37.465 0)
+    (property "Intersheetrefs" "${INTERSHEET_REFS}" (at 149.5604 37.465 0)
       (effects (font (size 1.27 1.27)) (justify left) hide)
     )
@@
     )
   )
+  (global_label "VBUS" (shape input) (at 219.71 40.005 180) (fields_autoplaced)
+    (effects (font (size 1.27 1.27)) (justify right))
+    (property "Intersheetrefs" "${INTERSHEET_REFS}" (at 212.4804 40.005 0)
+      (effects (font (size 1.27 1.27)) (justify right) hide)
+    )
+  )
   (global_label "SDSCK" (shape input) (at 121.92 120.015 180) (fields_autoplaced)
     (effects (font (size 1.27 1.27)) (justify right))
@@
     )
   )
+  (global_label "USB" (shape output) (at 229.87 47.625 270) (fields_autoplaced)
+    (effects (font (size 1.27 1.27)) (justify right))
+    (property "Intersheetrefs" "${INTERSHEET_REFS}" (at 229.87 53.766 90)
+      (effects (font (size 1.27 1.27)) (justify right) hide)
+    )
+  )
   (global_label "VBUS" (shape output) (at 276.225 65.405 0) (fields_autoplaced)
     (effects (font (size 1.27 1.27)) (justify left))
@@
     )
   )
+  (global_label "USB" (shape input) (at 42.545 48.26 180) (fields_autoplaced)
+    (effects (font (size 1.27 1.27)) (justify right))
+    (property "Intersheetrefs" "${INTERSHEET_REFS}" (at 36.404 48.26 0)
+      (effects (font (size 1.27 1.27)) (justify right) hide)
+    )
+  )
   (global_label "SDCD" (shape output) (at 121.92 130.175 180) (fields_autoplaced)
     (effects (font (size 1.27 1.27)) (justify right))
@@
     )
   )
+  (symbol (lib_id "power:GND") (at 222.25 47.625 0) (unit 1)
+    (in_bom yes) (on_board yes) (dnp no)
+    (property "Reference" "#PWR047" (at 222.25 53.975 0)
+      (effects (font (size 1.27 1.27)) hide)
+    )
+    (property "Value" "GND" (at 222.25 51.435 0)
+      (effects (font (size 1.27 1.27)))
+    )
+    (property "Footprint" "" (at 222.25 47.625 0)
+      (effects (font (size 1.27 1.27)) hide)
+    )
+    (property "Datasheet" "" (at 222.25 47.625 0)
+      (effects (font (size 1.27 1.27)) hide)
+    )
+    (pin "1")
+    (instances
+      (project "Watchy"
+        (path "/03039abc-65dd-445c-a352-9e386e1f31aa"
+          (reference "#PWR047") (unit 1)
+        )
+      )
+      (project "EPDBat"
+        (path "/46c350bb-7de4-4e81-aafd-4af55e37aab0"
+          (reference "#PWR036") (unit 1)
+        )
+      )
+      (project "Logger"
+        (path "/babeabf2-f3b0-4ed5-8d9e-0215947e6cf3"
+          (reference "#PWR044") (unit 1)
+        )
+      )
+    )
+  )
   (symbol (lib_id "Device:C") (at 119.38 158.115 0) (mirror y) (unit 1)
     (in_bom yes) (on_board yes) (dnp no)
@@
     )
   )
+  (symbol (lib_id "Device:R") (at 222.25 43.815 0) (unit 1)
+    (in_bom yes) (on_board yes) (dnp no)
+    (property "Reference" "R12" (at 222.25 43.815 90)
+      (effects (font (size 1.27 1.27)))
+    )
+    (property "Value" "100K 1%" (at 224.79 43.18 90)
+      (effects (font (size 1.27 1.27)))
+    )
+    (property "Footprint" "RevK:R_0402" (at 220.472 43.815 90)
+      (effects (font (size 1.27 1.27)) hide)
+    )
+    (property "Datasheet" "~" (at 222.25 43.815 0)
+      (effects (font (size 1.27 1.27)) hide)
+    )
+    (property "LCSC Part #" "C5139597" (at 222.25 43.815 90)
+      (effects (font (size 1.27 1.27)) hide)
+    )
+    (pin "1")
+    (pin "2")
+    (instances
+      (project "Watchy"
+        (path "/03039abc-65dd-445c-a352-9e386e1f31aa"
+          (reference "R12") (unit 1)
+        )
+      )
+      (project "EPDBat"
+        (path "/46c350bb-7de4-4e81-aafd-4af55e37aab0"
+          (reference "R16") (unit 1)
+        )
+      )
+      (project "Logger"
+        (path "/babeabf2-f3b0-4ed5-8d9e-0215947e6cf3"
+          (reference "R11") (unit 1)
+        )
+      )
+    )
+  )
   (symbol (lib_id "RevK:WS2812B-1mm") (at 27.305 158.115 0) (mirror x) (unit 1)
     (in_bom yes) (on_board yes) (dnp no)
@@
     )
   )
+  (symbol (lib_id "Transistor_FET:BSS83P") (at 227.33 40.005 0) (unit 1)
+    (in_bom yes) (on_board yes) (dnp no)
+    (property "Reference" "Q4" (at 234.823 38.608 90)
+      (effects (font (size 1.27 1.27)) (justify left))
+    )
+    (property "Value" "CJ2301" (at 232.791 43.307 90)
+      (effects (font (size 1.27 1.27)) (justify left))
+    )
+    (property "Footprint" "RevK:SOT-23" (at 232.41 41.91 0)
+      (effects (font (size 1.27 1.27) italic) (justify left) hide)
+    )
+    (property "Datasheet" "http://www.farnell.com/datasheets/1835997.pdf" (at 227.33 40.005 0)
+      (effects (font (size 1.27 1.27)) (justify left) hide)
+    )
+    (property "LCSC Part #" "C5224170" (at 227.33 40.005 90)
+      (effects (font (size 1.27 1.27)) hide)
+    )
+    (property "JLCPCB Rotation Offset" "180" (at 227.33 40.005 90)
+      (effects (font (size 1.27 1.27)) hide)
+    )
+    (pin "1")
+    (pin "2")
+    (pin "3")
+    (instances
+      (project "Watchy"
+        (path "/03039abc-65dd-445c-a352-9e386e1f31aa"
+          (reference "Q4") (unit 1)
+        )
+      )
+      (project "EPDBat"
+        (path "/46c350bb-7de4-4e81-aafd-4af55e37aab0"
+          (reference "Q2") (unit 1)
+        )
+      )
+      (project "Logger"
+        (path "/babeabf2-f3b0-4ed5-8d9e-0215947e6cf3"
+          (reference "Q3") (unit 1)
+        )
+      )
+    )
+  )
   (symbol (lib_id "power:PWR_FLAG") (at 173.355 29.845 0) (unit 1)
     (in_bom yes) (on_board yes) (dnp no) (fields_autoplaced)
@@
         )
       )
+    )
+  )
+  (symbol (lib_id "power:+3.3V") (at 229.87 34.925 0) (unit 1)
+    (in_bom yes) (on_board yes) (dnp no) (fields_autoplaced)
+    (property "Reference" "#PWR020" (at 229.87 38.735 0)
+      (effects (font (size 1.27 1.27)) hide)
+    )
+    (property "Value" "+3.3V" (at 229.87 30.7919 0)
+      (effects (font (size 1.27 1.27)))
+    )
+    (property "Footprint" "" (at 229.87 34.925 0)
+      (effects (font (size 1.27 1.27)) hide)
+    )
+    (property "Datasheet" "" (at 229.87 34.925 0)
+      (effects (font (size 1.27 1.27)) hide)
+    )
+    (pin "1")
+    (instances
+      (project "EPDBat"
+        (path "/46c350bb-7de4-4e81-aafd-4af55e37aab0"
+          (reference "#PWR020") (unit 1)
+        )
+      )
+      (project "Logger"
+        (path "/babeabf2-f3b0-4ed5-8d9e-0215947e6cf3"
+          (reference "#PWR043") (unit 1)
+        )
+      )
