File: PCB/Logger/Logger.kicad_sch (KiCad schematic)
At the start: 77 parts, among them J2 USB-C-Socket-V, J3 JST-PH-SM4-TB, J3 USB-PROG, J5 Conn_01x05, J6 TF_PUSH, J8 Shelly, Q1 C179347, Q4 CJ2301, U1 TP4054, U10 ESP32-S3-MINI-1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

Commit message: Extra ESD so GPIO0 can be used as a button
Parts:
- added D27: ~, RevK:DFN1006-2L, symbol RevK:ES05D1MC10
Connections:
- net GND: now also D27.2
- net at J8.2 (0), U10.4 (GPIO0): now also D27.1
Changed lines of the file:
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@@
   (junction (at 178.435 161.925) (diameter 0) (color 0 0 0 0)
   )
+  (junction (at 73.025 43.18) (diameter 0) (color 0 0 0 0)
+  )
   (junction (at 184.15 154.305) (diameter 0) (color 0 0 0 0)
   )
@@
     (stroke (width 0) (type default))
   )
+  (wire (pts (xy 73.025 43.18) (xy 83.82 43.18))
+    (stroke (width 0) (type default))
+  )
   (wire (pts (xy 92.075 161.925) (xy 97.79 161.925))
     (stroke (width 0) (type default))
@@
     )
   )
+  (symbol (lib_id "power:GND") (at 83.82 50.8 0) (unit 1)
+    (in_bom yes) (on_board yes) (dnp no) (fields_autoplaced)
+    (property "Reference" "#PWR011" (at 83.82 57.15 0)
+      (effects (font (size 1.27 1.27)) hide)
+    )
+    (property "Value" "GND" (at 83.82 55.2434 0)
+      (effects (font (size 1.27 1.27)))
+    )
+    (property "Footprint" "" (at 83.82 50.8 0)
+      (effects (font (size 1.27 1.27)) hide)
+    )
+    (property "Datasheet" "" (at 83.82 50.8 0)
+      (effects (font (size 1.27 1.27)) hide)
+    )
+    (pin "1")
+    (instances
+      (project "USBA"
+        (path "/2d210a96-f81f-42a9-8bf4-1b43c11086f3"
+          (reference "#PWR011") (unit 1)
+        )
+      )
+      (project "EPD75"
+        (path "/46c350bb-7de4-4e81-aafd-4af55e37aab0"
+          (reference "#PWR05") (unit 1)
+        )
+      )
+      (project "Logger"
+        (path "/babeabf2-f3b0-4ed5-8d9e-0215947e6cf3"
+          (reference "#PWR045") (unit 1)
+        )
+      )
+    )
+  )
   (symbol (lib_id "power:GND") (at 222.25 47.625 0) (unit 1)
     (in_bom yes) (on_board yes) (dnp no)
@@
         )
       )
+    )
+  )
+  (symbol (lib_id "RevK:ES05D1MC10") (at 83.82 46.99 90) (unit 1)
+    (in_bom yes) (on_board yes) (dnp no)
+    (property "Reference" "D27" (at 77.47 48.26 90)
+      (effects (font (size 1.27 1.27)) (justify right))
+    )
+    (property "Value" "~" (at 83.82 46.99 0)
+      (effects (font (size 1.27 1.27)))
+    )
+    (property "Footprint" "RevK:DFN1006-2L" (at 80.645 46.355 0)
+      (effects (font (size 1.27 1.27)) hide)
+    )
+    (property "Datasheet" "" (at 83.82 46.99 0)
+      (effects (font (size 1.27 1.27)) hide)
+    )
+    (property "LCSC Part #" "C5137770" (at 86.995 46.99 0)
+      (effects (font (size 1.27 1.27)) hide)
+    )
+    (pin "2")
+    (pin "1")
+    (instances
+      (project "EPD75"
+        (path "/46c350bb-7de4-4e81-aafd-4af55e37aab0"
+          (reference "D27") (unit 1)
+        )
+      )
+      (project "Logger"
+        (path "/babeabf2-f3b0-4ed5-8d9e-0215947e6cf3"
+          (reference "D24") (unit 1)
+        )
+      )

Commit message: FFS USB not working
Connections:
- net +3.3V: now also Q4.2 (S); no longer Q4.3 (D)
- net USB: now also Q4.3 (D); no longer Q4.2 (S)
Changed lines of the file:
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@@
     )
   )
-  (symbol (lib_id "Transistor_FET:BSS83P") (at 227.33 40.005 0) (unit 1)
+  (symbol (lib_id "Transistor_FET:BSS83P") (at 227.33 40.005 0) (mirror x) (unit 1)
     (in_bom yes) (on_board yes) (dnp no)
-    (property "Reference" "Q4" (at 234.823 38.608 90)
+    (property "Reference" "Q4" (at 234.823 41.402 90)
       (effects (font (size 1.27 1.27)) (justify left))
     )
-    (property "Value" "CJ2301" (at 232.791 43.307 90)
+    (property "Value" "CJ2301" (at 232.791 36.703 90)
       (effects (font (size 1.27 1.27)) (justify left))
     )
-    (property "Footprint" "RevK:SOT-23" (at 232.41 41.91 0)
+    (property "Footprint" "RevK:SOT-23" (at 232.41 38.1 0)
       (effects (font (size 1.27 1.27) italic) (justify left) hide)
     )
-    (property "Datasheet" "http://www.farnell.com/datasheets/1835997.pdf" (at 227.33 40.005 0)
+    (property "Datasheet" "" (at 227.33 40.005 0)
       (effects (font (size 1.27 1.27)) (justify left) hide)
     )

Commit message: New headers
Parts:
- removed J3: USB-PROG, RevK:USB-PROG, symbol RevK:USB-PROG
- removed J8: Shelly, RevK:Shelly, symbol RevK:Shelly
- added J4: Reset, RevK:AA-Pad, symbol Connector_Generic:Conn_01x02
- added J7: TC2030-USB-NL-DS, RevK:Tag-Connect_TC2030-IDC-NL_2x03_P1.27mm_Vertical, symbol RevK:TC2030-USB-NL
Connections:
- net D+: now also J7.4 (D+)
- net D-: now also J7.3 (D-)
- net GND: now also U10.20 (GPIO16), U10.21 (GPIO17), U10.22 (GPIO18), J4.1 (Pin_1), J7.5 (GND), J7.6 (GND)
- net VBUS: now also J7.1 (VBUS), J7.2 (VBUS)
- net at U10.25 (GPIO21): now also J4.2 (Pin_2)
- no-connect marks 25 -> 24

Commit message: Resistors
Parts:
- added R15, R16, R17, R18, R19, R20: 10K, RevK:R_0402, symbol Device:R
Connections:
- net +3.3V: now also J6.4 (VDD), R15.1, R16.1, R17.1, R18.1, R19.1, R20.1
- net SDMISO: now also R16.2
- net SDMOSI: now also R18.2
- net SDSCK: now also R17.2
- net SDSS: now also R19.2
- net SPWR: no longer J6.4 (VDD)
- net at J6.1 (DAT2): now also R20.2
- net at J6.8 (DAT1): now also R15.2
- no-connect marks 24 -> 22
Other:
- moved on the sheet: D27, J5, J6
